File: aardvark-qwiic-adapter.kicad_pcb (KiCad board)
At the start: 2 copper layers, 22.9 x 20.3 mm, 7 parts, among them J1 Conn_02x05_Odd_Even, J2 Conn_01x04, J3 Conn_01x04, J4 Conn_01x02, U1 AP7361C-33E

Commit message: Connect +3.3V
Routing:
- net +3.3V: track 2.63 -> 10.2 mm
- net /GPIO02: track 27.2 -> 26.4 mm
Changed lines of the file:
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@@
   (segment (start 127 90.0938) (end 124.841 87.9348) (width 0.25) (layer "B.Cu") (net 3))
   (segment (start 131.783299 82.455) (end 133.445 82.455) (width 0.25) (layer "B.Cu") (net 3))
+  (segment (start 126.243 92.4052) (end 128.4042 90.244) (width 0.25) (layer "F.Cu") (net 4))
   (segment (start 127.155 85.9256) (end 127.155 84.43) (width 0.25) (layer "F.Cu") (net 4))
+  (segment (start 128.4042 90.244) (end 128.4042 87.2562) (width 0.25) (layer "F.Cu") (net 4))
+  (segment (start 128.143 86.995) (end 127 86.995) (width 0.25) (layer "F.Cu") (net 4))
   (segment (start 127 86.0806) (end 127.155 85.9256) (width 0.25) (layer "F.Cu") (net 4))
+  (segment (start 128.4042 87.2562) (end 128.143 86.995) (width 0.25) (layer "F.Cu") (net 4))
   (segment (start 127 86.995) (end 127 86.0806) (width 0.25) (layer "F.Cu") (net 4))
+  (segment (start 120.1166 86.36) (end 116.84 86.36) (width 0.25) (layer "F.Cu") (net 5))
+  (segment (start 121.0564 87.2998) (end 120.1166 86.36) (width 0.25) (layer "F.Cu") (net 5))
+  (segment (start 132.08 86.36) (end 130.7084 86.36) (width 0.25) (layer "F.Cu") (net 5))
+  (segment (start 129.0828 87.9856) (end 129.0828 91.9154) (width 0.25) (layer "F.Cu") (net 5))
   (segment (start 121.0564 91.8718) (end 121.0564 87.2998) (width 0.25) (layer "F.Cu") (net 5))
-  (segment (start 120.1166 86.36) (end 116.84 86.36) (width 0.25) (layer "F.Cu") (net 5))
-  (segment (start 129.4892 86.36) (end 128.8542 86.995) (width 0.25) (layer "F.Cu") (net 5))
+  (segment (start 129.0828 91.9154) (end 127.1308 93.8674) (width 0.25) (layer "F.Cu") (net 5))
   (segment (start 123.052 93.8674) (end 121.0564 91.8718) (width 0.25) (layer "F.Cu") (net 5))
+  (segment (start 130.7084 86.36) (end 129.0828 87.9856) (width 0.25) (layer "F.Cu") (net 5))
   (segment (start 127.1308 93.8674) (end 123.052 93.8674) (width 0.25) (layer "F.Cu") (net 5))
-  (segment (start 128.8542 86.995) (end 128.8542 92.144) (width 0.25) (layer "F.Cu") (net 5))
-  (segment (start 121.0564 87.2998) (end 120.1166 86.36) (width 0.25) (layer "F.Cu") (net 5))
-  (segment (start 128.8542 92.144) (end 127.1308 93.8674) (width 0.25) (layer "F.Cu") (net 5))
-  (segment (start 132.08 86.36) (end 129.4892 86.36) (width 0.25) (layer "F.Cu") (net 5))
   (segment (start 120.3452 92.4306) (end 120.3452 89.281) (width 0.25) (layer "F.Cu") (net 6))
   (segment (start 130.0734 92.075) (end 127.831 94.3174) (width 0.25) (layer "F.Cu") (net 6))
